File: PCB/eink.kicad_pcb (KiCad board)
At the start: 2 copper layers, 44.6 x 96 mm, 68 parts, among them J1 USB_C_Receptacle_USB2.0_14P, J5 Battery, J6 Micro_SD_Card, Q1 AO3401A, Q3 Si1308EDL, SW1 BOOTSEL, SW2 RST, SW4 SW_MEC_5E, U1 RP2040, U2 MCP1700x-300xxTT, U3 W25Q16JVZPIQ TR, U4 MCP73831-2-OT, Y1 12 MHz

Commit message: Add files via upload
Parts:
- removed the C20 at (219.2, 52.3)
- removed FPC24PIN_0.5mm1: E-Ink_Disp, Connector_FFC-FPC:Amphenol_F32Q-1A7x1-11024_1x24-1MP_P0.5mm_Horizontal
- removed J5: Battery, Connector_JST:JST_EH_S2B-EH_1x02_P2.50mm_Horizontal
- removed J6: Micro_SD_Card, Connector_Card:microSD_HC_Hirose_DM3D-SF
- removed the R11 at (223.4, 64.9)
- removed the R12 at (230.4, 64.9)
- removed the R13 at (223.4, 63.8)
- removed the R15 at (226.9, 64.9)
- removed R17: 10K, Resistor_SMD:R_0402_1005Metric
- removed SW4: SW_MEC_5E, Button_Switch_SMD:KEY-SMD_4P-L4.7-W3.5_EVQ9P
- added C3: 10uF, Capacitor_SMD:C_0603_1608Metric, F.Cu at (216.7, 69.8)
- added CN1: Battery, Connector_JST:CONN-SMD_2P-P2.00_PH2.0-SPWB, F.Cu at (194.9, 129.7)
- added R3: 10K, Resistor_SMD:R_0402_1005Metric, F.Cu at (224.7, 93.4)
- added R4: 10K, Resistor_SMD:R_0402_1005Metric, F.Cu at (226.7, 93.4)
- added R5: 10K, Resistor_SMD:R_0402_1005Metric, F.Cu at (228.7, 93.4)
- added SD-CARD1: ~, Connector_Card:TF-SMD_TF-015, F.Cu at (225.4, 79.3)
- added SW3: ~, Button_Switch_SMD:SW-SMD_EVQPUD02K-1, F.Cu at (192.3, 77.8)
- added U5: ~, Connector_FFC-FPC:FPC-SMD_24P-P0.50_YUANDI_FPC-0.5FX-24PH20, F.Cu at (212.3, 128.9)
- SW1: value BOOTSEL -> ~; footprint Button_Switch_SMD:SW_SPST_TS-1088-xR020 -> Button_Switch_SMD:SW-SMD_EVQPUD02K-1
- SW2: value RST -> ~; footprint Button_Switch_SMD:SW_SPST_TS-1088-xR020 -> Button_Switch_SMD:SW-SMD_EVQPUD02K-1
- moved SW2 32.8 mm to (192.3, 85.0), turned to 180 degrees
- moved C1 28.5 mm to (191.6, 103.4)
- moved D1 28.5 mm to (198.3, 104.0)
- moved R6 28.5 mm to (197.8, 105.4)
- moved R7 28.5 mm to (191.6, 105.3)
- moved U1 28.5 mm to (194.7, 104.4)
- moved SW1 12.9 mm to (192.3, 70.1), turned to 180 degrees
- moved R15 10.7 mm to (208.7, 123.6)
- moved C20 10.7 mm to (207.5, 113.2)
- moved C21 10.7 mm to (217.1, 114.3)
- moved C22 10.7 mm to (220.7, 125.3)
- moved C23 10.7 mm to (213.4, 123.2)
- moved D3 10.7 mm to (218.3, 115.7)
- moved D4 10.7 mm to (218.3, 113.0)
- moved D5 10.7 mm to (220.3, 123.5)
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- renumbered C17 to C1, C1 to C10, C2 to C11, C3 to C12, C15 to C13, C16 to C14, C4 to C15, C5 to C16, C6 to C17, C7 to C18, C8 to C19, C18 to C2, C28 to C20, C29 to C21, C30 to C22, C22 to C23, C23 to C24, C31 to C25, C24 to C26, C25 to C27, C26 to C28, C21 to C29, C27 to C30, C13 to C4, C19 to C5, C10 to C6, C14 to C7, C11 to C8, C12 to C9, D6 to D2, D5 to D3, D3 to D5, Q3 to Q2, R4 to R10, R14 to R11, R6 to R12, R7 to R13, R5 to R14, R23 to R15, R8 to R6, R9 to R7, R10 to R8, R3 to R9, U4 to U1, U1 to U3, U3 to U4
Connections:
- C5 pad 2: Net-(U1-RUN) -> Net-(U3-RUN)
- R11 pad 2: Net-(U1-RUN) -> Net-(U3-RUN)
- R12 pad 2: Net-(R6-Pad2) -> Net-(R12-Pad2)
- SW1 pad 2: Net-(R6-Pad2) -> GPIO5
- SW2 pad 2: Net-(U1-RUN) -> Net-(U3-RUN)
- U3 pad 26: Net-(U1-RUN) -> Net-(U3-RUN)
- U3 pad 29: /Eink SCLK -> GPIO18
- U3 pad 30: /SDI -> GPIO19
Routing:
- net GPIO21: track 72.2 -> 0.00 mm, vias 2 -> 0
- net GPIO18: track 0.00 -> 71.3 mm, vias 0 -> 2
- net GPIO20: track 70.7 -> 0.00 mm, vias 2 -> 0
- net GPIO19: track 0.00 -> 69.5 mm, vias 0 -> 4
- net GPIO22: track 62.9 -> 0.00 mm, vias 2 -> 0
- net GPIO23: track 62.5 -> 0.00 mm, vias 2 -> 0
- net GPIO24: track 57.8 -> 0.00 mm, vias 2 -> 0
- net GPIO16: track 0.00 -> 49.4 mm, vias 0 -> 4
- net Net-(U3-RUN): track 0.00 -> 49.1 mm, vias 0 -> 2
- net /SDI: track 42.5 -> 0.00 mm, vias 2 -> 0
- net /Eink SCLK: track 40.7 -> 0.00 mm, vias 2 -> 0
- net Net-(U1-RUN): track 39.6 -> 0.00 mm
- net +3.3V: track 175.9 -> 143.3 mm
- net VBUS: track 105.7 -> 77.2 mm
- net Net-(R12-Pad2): track 0.00 -> 26.3 mm, vias 0 -> 2
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Other:
- board size 44.6 x 96 mm -> 44.6 x 85.1 mm

Commit message: Add files via upload
Parts:
- L1: footprint Inductor_SMD:L_6.3x6.3_H3 -> Inductor_SMD:L_Cenker_CKCS5020
Routing:
- net Net-(D5-A): track 21.2 -> 22.8 mm
- net GND: vias 242 -> 241
